File: psense.sch (KiCad schematic (older format))
At the start: 33 parts, among them J1 USB-micro-b, U1 PAC1720, U2 MCP2221A

Commit message: Layout done
Parts:
- removed R6: 10K, symbol R
- removed TP10: GP0, symbol TEST
- removed TP12: GP1, symbol TEST
- removed TP13: ~RST, symbol TEST
- removed TP14: URx, symbol TEST
- removed TP15: UTx, symbol TEST
- removed TP16: GP2, symbol TEST
- removed TP17: ~ALERT, symbol TEST
- C1: renamed from 10µF1; footprint (none) -> kicadlib:SMD_0603_C
- C2: renamed from C1; footprint (none) -> kicadlib:SMD_0603_C
- C3: renamed from C2; footprint (none) -> kicadlib:SMD_0603_C
- D1: footprint (none) -> kicadlib:SMD_0603_LED_REVERSED
- J1: footprint (none) -> kicadlib:usb_micro_b_smt
- R1, R2, R3, R4: footprint (none) -> kicadlib:SMD_0603_R
- R5: value R -> 10K; footprint (none) -> kicadlib:SMD_0603_R
- R6: renamed from R7; footprint (none) -> kicadlib:SMD_0603_R
- R7: renamed from R8; footprint (none) -> kicadlib:SMD_0603_R
- R8: renamed from R9; footprint (none) -> kicadlib:SMD_0603_R
- TP1, TP5, TP6: footprint (none) -> kicadlib:TEST_0.100
- TP10: renamed from TP11; footprint (none) -> kicadlib:TEST_0.100
- TP2: value S1_SELECT_HIGH -> S1_SEL_H; footprint (none) -> kicadlib:TEST_0.100
- TP3: value S1_SELECT_LOW -> S1_SEL_L; footprint (none) -> kicadlib:TEST_0.100
- TP4: value S1_SELECT_COMMON -> S1_SEL_C; footprint (none) -> kicadlib:TEST_0.100
- TP7: value S2_SELECT_HIGH -> S2_SEL_H; footprint (none) -> kicadlib:TEST_0.100
- TP8: value S2_SELECT_LOW -> S2_SEL_L; footprint (none) -> kicadlib:TEST_0.100
- TP9: value S2_SELECT_COMMON -> S2_SEL_C; footprint (none) -> kicadlib:TEST_0.100
- U1: footprint (none) -> kicadlib:SMD_10-DFN
- U2: footprint (none) -> kicadlib:SMD_14-SOIC
Connections:
- net GND: no longer R5.2
- net USB_VBUS: now also R5.2
- net ~RST: now also R5.1
- net ADDR_SEL: now reaches U1.6 (ADDR_SEL)
- net ADDR_SEL: no longer R5.1
- net ~ALERT: now reaches U1.7 (~ALERT)
- net VUSB: now reaches C3.2, U2.11 (VUSB)
- net GP3: now reaches D1.1 (K), U2.8 (GP3)
- no-connect marks 2 -> 9
Other:
- note removed: "Test Breakouts"
- note removed: "nopop"
- moved on the sheet: C1, D1, R6
