File: psense.kicad_pcb (KiCad board)
At the start: 2 copper layers, 39.4 x 20.3 mm, 25 parts, among them J1 USB-micro-b, U1 PAC1720, U2 MCP2221A

Commit message: Tidy up a bit
Parts:
- moved C2 0.25 mm to (173.4, 117.7)
- moved C3 0.25 mm to (168.3, 117.7)
Other:
- board text added: "psense v1"
- board text removed: "psense v1.0"
Changed lines of the file:
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@@
     (links 43)
     (no_connects 6)
-    (area 157.061 101.26 199.518334 122.36)
+    (area 158.039999 101.524999 197.560001 121.995001)
     (thickness 1.6)
-    (drawings 13)
+    (drawings 11)
     (tracks 113)
     (zones 0)
@@
   )
   (module kicadlib:SMD_0603_C (layer F.Cu)
-    (at 173.355 117.475)
+    (at 173.355 117.729)
     (fp_text reference C2 (at 1.27 0) (layer F.SilkS)
       (effects (font (size 0.75 0.75) (thickness 0.12)))
@@
   )
   (module kicadlib:SMD_0603_C (layer F.Cu)
-    (at 168.275 117.475)
+    (at 168.275 117.729)
     (fp_text reference C3 (at 1.27 0) (layer F.SilkS)
       (effects (font (size 0.75 0.75) (thickness 0.12)))
@@
     (effects (font (size 1 1) (thickness 0.15)) (justify left))
   )
-  (gr_text "psense v1.0" (at 159.385 102.87) (layer F.Mask)
-    (effects (font (size 1 1) (thickness 0.15)) (justify left))
-  )
-  (gr_text github.com/noahp/psense (at 159.385 120.015) (layer F.Cu)
-    (effects (font (size 1 1) (thickness 0.15)) (justify left))
-  )
-  (gr_text "psense v1.0" (at 159.385 102.87) (layer F.Cu)
+  (gr_text "psense v1" (at 159.385 102.87) (layer F.Mask)
     (effects (font (size 1 1) (thickness 0.15)) (justify left))
   )
@@
     (effects (font (size 0.75 0.75) (thickness 0.12)))
   )
+  (segment (start 171.831 116.169) (end 171.831 117.729) (width 0.25) (layer F.Cu) (net 1))
   (segment (start 163.02 110.46) (end 164.604998 110.46) (width 0.25) (layer F.Cu) (net 1))
   (segment (start 164.604998 110.46) (end 166.404999 108.659999) (width 0.25) (layer F.Cu) (net 1))
@@
   (segment (start 176.276 117.475) (end 174.371 115.57) (width 0.25) (layer F.Cu) (net 1))
   (segment (start 177.673 106.045) (end 171.704 106.045) (width 0.25) (layer F.Cu) (net 1))
-  (segment (start 171.831 117.475) (end 171.831 116.169) (width 0.25) (layer F.Cu) (net 1))
   (segment (start 171.831 116.169) (end 172.43 115.57) (width 0.25) (layer F.Cu) (net 1))
   (segment (start 172.43 115.57) (end 172.88 115.57) (width 0.25) (layer F.Cu) (net 1))
@@
   (segment (start 167.386 106.045) (end 167.386 107.856) (width 0.25) (layer F.Cu) (net 24))
   (segment (start 167.386 107.856) (end 167.48 107.95) (width 0.25) (layer F.Cu) (net 24))
-  (segment (start 168.275 117.475) (end 168.275 117.275) (width 0.25) (layer F.Cu) (net 25))
-  (segment (start 168.275 117.275) (end 168.555001 116.994999) (width 0.25) (layer F.Cu) (net 25))
-  (segment (start 168.555001 116.994999) (end 168.555001 112.385001) (width 0.25) (layer F.Cu) (net 25))
+  (segment (start 168.555001 112.385001) (end 168.555001 116.748999) (width 0.25) (layer F.Cu) (net 25))
+  (segment (start 168.555001 116.748999) (end 168.275 117.029) (width 0.25) (layer F.Cu) (net 25))
+  (segment (start 168.275 117.029) (end 168.275 117.729) (width 0.25) (layer F.Cu) (net 25))
   (segment (start 168.555001 112.385001) (end 167.93 111.76) (width 0.25) (layer F.Cu) (net 25))
   (segment (start 167.93 111.76) (end 167.48 111.76) (width 0.25) (layer F.Cu) (net 25))

Commit message: Fix https://github.com/noahp/psense/issues/1 https://github.com/noahp/psense/issues/2 https://github.com/noahp/psense/issues/3
Parts:
- C1: value 10µF -> 0.1µF
- J1: footprint kicadlib:usb_micro_b_smt -> kicadlib:SMD_MICRO_USB_B_WPEGS
- moved J1 0.51 mm to (159.5, 111.8)
Routing:
- net /I2C_SCL: track 16.1 -> 17.8 mm, vias 0 -> 2
- net /USB_VBUS: track 47.6 -> 48.3 mm, vias 0 -> 2
Other:
- board text added: "psense v2"
- board text removed: "psense v1"

Commit message: Use FT200XD instead
Parts:
- removed D1: I2C ACTIVE LED, kicadlib:SMD_0603_LED_REVERSED
- removed R7, R8: 4.7K, kicadlib:SMD_0603_R
- C2: value 10µF -> 10pF; footprint kicadlib:SMD_0603_C -> Capacitor_SMD:C_0603_1608Metric
- C3: value 0.22-0.47µF -> 100nF; footprint kicadlib:SMD_0603_C -> Capacitor_SMD:C_0603_1608Metric
- J1: value USB-micro-b -> USB_B_Micro; footprint kicadlib:SMD_MICRO_USB_B_WPEGS -> Connector_USB:USB_Micro-B_Molex_47346-0001
- R5: value 10K -> 1K; footprint kicadlib:SMD_0603_R -> Resistor_SMD:R_0603_1608Metric
- R6: footprint kicadlib:SMD_0603_R -> Resistor_SMD:R_0603_1608Metric
- U2: value MCP2221A -> FT200XD; footprint kicadlib:SMD_14-SOIC -> Package_DFN_QFN:DFN-10-1EP_3x3mm_P0.5mm_EP1.55x2.48mm
- moved C2 35.9 mm to (145.9, 94.6)
- moved R5 31.0 mm to (153.7, 92.7), turned to 0 degrees
- moved C3 26.3 mm to (145.4, 104.8)
- moved U2 13.7 mm to (173.4, 98.4), turned to 0 degrees
- moved R6 13.1 mm to (163.8, 94.6), turned to 0 degrees
- moved J1 1.31 mm to (160.7, 111.1)
Connections:
- net /URx renamed Net-(U2-Pad5)
- C3 pad 1: GND -> /FT200XD_VCCIO
- C3 pad 2: /VUSB -> GND
- R5 pad 1: /~RST -> /FT200XD_VCCIO
- R5 pad 2: /USB_VBUS -> /I2C_SCL
- R6 pad 1: /USB_VBUS -> /FT200XD_VCCIO
- R6 pad 2: Net-(D1-Pad2) -> /I2C_SDA
- U2 pad 1: /USB_VBUS -> /USB_DM
- U2 pad 10: /I2C_SCL -> /USB_DP
- U2 pad 11: /VUSB -> GND
- U2 pad 2: /GP0 -> /FT200XD_VCCIO
- U2 pad 3: /GP1 -> /FT200XD_VCCIO
- U2 pad 4: /~RST -> /USB_VBUS
- U2 pad 6: /UTx -> /I2C_SCL
- U2 pad 7: /GP2 -> /FT200XD_VCCIO
- U2 pad 8: /GP3 -> /I2C_SDA
- U2 pad 9: /I2C_SDA -> GND
Routing:
- net /USB_VBUS: track 48.3 -> 0.00 mm, vias 2 -> 0
- net /I2C_SCL: track 17.8 -> 0.00 mm, vias 2 -> 0
- net /I2C_SDA: track 16.7 -> 0.00 mm
- net /VUSB: track 6.79 -> 0.00 mm
- net /USB_DP: track 5.51 -> 0.00 mm
- net /USB_DM: track 5.26 -> 0.00 mm
- net /~RST: track 3.36 -> 0.00 mm
- net /GP3: track 1.94 -> 0.00 mm
- net Net-(D1-Pad2): track 1.27 -> 0.00 mm
Other:
- board text added: "psense v3"
- board text removed: "I2C ACTIVE"
- board text removed: "psense v2"
